File: kicad_psu.kicad_pcb (KiCad board)
At the start: 2 copper layers, 35.6 x 55.9 mm, 17 parts, among them J1 Barrel_Jack_Switch, J2 Conn_01x03_Pin, J3 Conn_01x03_Pin, J4 Conn_01x02_Pin, J5 Screw_Terminal_01x02, J6 Conn_01x02_Pin, J7 Screw_Terminal_01x02, U1 LM7805_TO220, U2 LM317_TO-220

Commit message: Finished PSU without logos
Parts:
- moved J2 132.0 mm to (80.7, 64.1), turned to 90 degrees
- moved C2 130.4 mm to (77.5, 73.0)
- moved U1 126.7 mm to (83.2, 77.8), turned to 180 degrees
- moved D1 126.7 mm to (94.3, 87.0)
- moved C1 124.6 mm to (82.6, 73.0)
- moved U2 117.8 mm to (78.1, 98.7)
- moved S1 117.1 mm to (95.1, 75.6), turned to 180 degrees
- moved R3 116.5 mm to (90.2, 96.5)
- moved J5 111.0 mm to (91.4, 66.7)
- moved J1 109.6 mm to (89.2, 87.3)
- moved C3 109.6 mm to (81.3, 103.5)
- moved R1 109.3 mm to (97.8, 93.3), turned to 180 degrees
- moved R2 106.8 mm to (97.8, 99.7), turned to 180 degrees
- moved J3 93.7 mm to (80.7, 114.3), turned to 90 degrees
- moved J7 77.6 mm to (96.5, 111.8), turned to 180 degrees
Routing:
- net /3V3: track 0.00 -> 75.2 mm
- net /5V: track 0.00 -> 58.1 mm
- net /12V: track 0.00 -> 45.5 mm
- net Net-(U2-ADJ): track 0.00 -> 30.6 mm
- net /PWR_out1: track 0.00 -> 22.7 mm
- net /PWR_out2: track 0.00 -> 21.7 mm
- net /PWR_input: track 0.00 -> 20.4 mm
- net Net-(D1-A): track 0.00 -> 6.77 mm
- added copper zone on B.Cu, net GND
Other:
- board size 35.6 x 55.9 mm -> 30.5 x 54 mm
